Commit message: tracker

File: src/urdf/lexus_rx_450h_description/urdf/navi_car.urdf (robot description, URDF)
Before this commit: robot navi_car, 3 links, 2 joints
Links:
- added link gnss
- added link imu
Joints:
- added joint gnss_joint: type fixed, parent base_link, child gnss, origin xyz=0 0 0 rpy=0 0 0
- added joint imu_joint: type fixed, parent base_link, child imu, origin xyz=0 0 0 rpy=0 0 0

Commit message: fix bug for imu zyx rotation

File: src/urdf/lexus_rx_450h_description/urdf/navi_car.urdf (robot description, URDF)
Before this commit: robot navi_car, 3 links, 2 joints
Links:
- removed link nav_base
- added link axis, mass 0.25; collision box size=0.25 0.4 0.6; visual cylinder length=0.3 radius=0.2
- link base_link: mass 0.25 -> None; geometry visual cylinder length=0.05 radius=0.05
- link lidar_front: mass 0.1 -> None
Joints:
- removed joint nav_base_joint
- added joint axis_joint: type continuous, parent base_link, child axis, origin xyz=0 0 0 rpy=0 0 0
- joint lidar_front_joint: parent base_link -> axis

Commit message: real obj tracking + prediction

File: src/urdf/lexus_rx_450h_description/urdf/navi_car.urdf (robot description, URDF)
Before this commit: robot navi_car, 3 links, 2 joints
Links:
- added link nav_base
Joints:
- added joint nav_base_joint: type fixed, parent base_link, child nav_base, origin xyz=0 0 0 rpy=0 0 0
